File: Boards/DP8473/DP8473_v11.kicad_sch (KiCad schematic)
At the start: 38 parts, among them J1 Power, J2 PWM 7-0, J3 Digital, J4 128x64 monochrome LCD, parall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, J5 FDD A: B:, J5 FDD C: D:, J7 PS/2 keyboard, J8 DE9 male - to null modem (twi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, P1 2k2, Q1 24 MHz, Q2 BC547, Q3 BC557, SW1 RESET, U1 DP8473

Commit message: Build 26th of May 2025 changes:
- UI with LCD output now doesn't require a physical keyboard,
- TYPEINTO command opens files with append instead of truncate,
- bugfix in the DELAY_MS macro,
- DP8473 Kicad schematic parts numbers reordered to match the Eagle PCB.
Parts:
- added C11: 100n, Capacitor_THT:C_Disc_D7.5mm_W2.5mm_P5.00mm, symbol Device:C
- renumbered C2 to C1, C3 to C10, C2 to C3, C2 to C4, C1 to C5, C2 to C6, C5 to C8, C4 to C9-C7, U1 to IC1, J5 to J6, JP1 to JP2, R7-R11 to R1-R5, R1 to R10, R2 to R11, P1 to R12, R5 to R7, R3 to R8, R4 to R9, JP1 to SW1.1, JP1 to SW1.2
Connections:
- net +5V: now also C11.1
- net GND: now also C11.2
Other:
- note added: "Configuration"
- note added: "JP1 (FDD A: B:) JP2 (FDD C: D:) Pin 2 behavior: 1-2: density select 2-3: 8" TG43 line"
- note added: "SW1.1 UI config: 1-2: LCD + keyboard 2-3: serial/USB only"
- note added: "SW1.2 baud rate: 1-2: 115200 bps 2-3: 9600 bps"
- note removed: "Configuration jumpers"
- note removed: "JP1 UI config: 1-2: LCD + keyboard 2-3: serial/USB only"
- note removed: "JP2 baud rate: 1-2: 115200 bps 2-3: 9600 bps"
- note removed: "JP3 (FDD A: B:) JP4 (FDD C: D:) Pin 2 behavior: 1-2: density select 2-3: 8" TG43 line"
- moved on the sheet: C10, C9-C7
